File: tsal-r-ckctan.kicad_pcb (KiCad board)
At the start: 2 copper layers, 100 x 86 mm, 50 parts, among them J1 Conn_01x02_Pin, J2 Conn_01x02_Pin, U1 TL431, U2 LTV-817, U3 B1212, U4 2N7002, U5 2N7002, U6 NCE60P04R, U7 NE555

Commit message: Add files via upload
Parts:
- removed U1: TL431, Final Project:P8
- added U8: TL431DBZ, Package_TO_SOT_SMD:SOT-23, F.Cu at (38.7, 97.1)
- D3: footprint LED_SMD:LED_0805_2012Metric -> LED_SMD:LED_0805_2012Metric_Pad1.15x1.40mm_HandSolder
Routing:
- net /Vref: track 27.2 -> 32.4 mm
- net Net-(U8-REF): track 16.4 -> 11.5 mm
- net GND: track 157.1 -> 159.7 mm

Commit message: Add files via upload
Parts:
- D3: footprint LED_SMD:LED_0805_2012Metric_Pad1.15x1.40mm_HandSolder -> LED_SMD:LED_0805_2012Metric
- moved Conn_01x1 14.8 mm to (122.1, 75.3)
- moved R_LED1 9.63 mm to (108.4, 71.8)
- moved R19 8.78 mm to (122.0, 64.0)
- moved H2 7.82 mm to (123.3, 100.2)
- moved H4 7.82 mm to (30.4, 100.2)
- moved D1 6.97 mm to (59.5, 57.0)
- moved J2 6.97 mm to (40.0, 61.2)
- moved R8 6.97 mm to (50.2, 61.3)
- moved R9 6.97 mm to (46.4, 61.3)
- moved C4 6.81 mm to (72.3, 98.4)
- moved R15 6.38 mm to (91.1, 43.5)
- moved C1 6.01 mm to (42.9, 95.0)
- moved R2 5.83 mm to (35.9, 95.0)
- moved R1 4.97 mm to (35.9, 89.7)
- moved R10 4.61 mm to (45.5, 86.0), turned to 90 degrees
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Routing:
- net GND: track 159.7 -> 132.6 mm
- net GLV+: track 31.3 -> 11.4 mm, vias 2 -> 5
- net /Vref: track 32.4 -> 16.9 mm
- net /RED+: track 45.5 -> 34.1 mm
- net VCC: track 170.7 -> 161.7 mm
- net Net-(U4-D): track 37.1 -> 29.6 mm
- net GLV-: track 88.0 -> 94.2 mm
- net /Vin: track 79.2 -> 84.0 mm
- net +12V: track 92.3 -> 88.0 mm
- net Net-(U8-REF): track 11.5 -> 7.21 mm
- net Net-(LM1--): track 22.6 -> 26.8 mm
- net Net-(R_LED1-K): track 8.19 -> 5.14 mm
- net Net-(U7-Q): track 9.76 -> 7.61 mm
- net Net-(LM1-+): track 18.8 -> 20.9 mm
- net Net-(J1-Pin_2): track 8.38 -> 10.4 mm
Other:
- board size 100 x 86 mm -> 100.1 x 79.3 mm

Commit message: Add files via upload
Parts:
- removed U5: 2N7002, Final Project:SOT-23TO-236_318-08_ONS
- removed U6: NCE60P04R, Final Project:DPAK_6020AK_WUX
- added Q1: MMBT3904, Package_TO_SOT_SMD:SOT-23, F.Cu at (96.4, 50.2)
- added Q2: AO3401A, Package_TO_SOT_SMD:SOT-23, F.Cu at (115.8, 50.2)
- moved R20 9.51 mm to (111.1, 50.0)
- moved R21 9.40 mm to (91.0, 50.0)
- moved R19 8.07 mm to (107.1, 50.0)
- moved D3 7.61 mm to (104.2, 50.0), turned to 90 degrees
- moved R18 5.64 mm to (101.3, 50.0)
- moved C8 3.90 mm to (116.0, 39.3), turned to -90 degrees
- moved R7 3.59 mm to (65.0, 31.1)
- moved R16 2.75 mm to (107.7, 39.3)
- moved R6 2.69 mm to (60.7, 31.1)
- moved U4 2.30 mm to (93.5, 65.9)
- moved R17 2.07 mm to (111.6, 39.3), turned to 90 degrees
- moved R5 1.70 mm to (56.3, 31.1)
- moved R3 0.89 mm to (52.0, 31.1)
- moved R15 0.71 mm to (91.0, 44.2)
Routing:
- net VCC: track 161.7 -> 126.9 mm, vias 0 -> 4
- net Net-(U7-Q): track 7.61 -> 39.1 mm
- net GLV-: track 94.2 -> 66.5 mm
- net GLV+: track 11.4 -> 37.4 mm, vias 5 -> 0
- net Net-(U7-THR): track 42.9 -> 27.7 mm, vias 0 -> 2
- net Net-(Q1-C): track 28.6 -> 19.4 mm
- net Net-(U7-CV): track 11.8 -> 18.9 mm
- net /RED+: track 34.1 -> 39.7 mm
- net Net-(U4-G): track 15.2 -> 12.9 mm
- net Net-(D3-K): track 5.43 -> 3.67 mm
- net /Vin: track 84.0 -> 85.5 mm
- net Net-(R5-Pad2): track 1.65 -> 2.59 mm
- net Net-(R6-Pad1): track 1.57 -> 2.48 mm
- net Net-(R3-Pad2): track 1.64 -> 2.46 mm
- net Net-(Q1-B): track 7.37 -> 7.03 mm, vias 0 -> 2
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- added copper zone on F.Cu, net GLV-
- removed copper zone on F.Cu, net GLV+
